Commit message: wheel description

File: src/alohamini_description/urdf/alohamini2pro_kinematic.urdf (robot description, URDF)
Before this commit: robot alohamini2pro_kinematic, 31 links, 30 joints
Joints:
- joint wheel1_joint: origin xyz=-0.1337 0.076522 0.063355 rpy=3.3411E-05 1.5707 2.618 -> xyz=-0.130229464 0.074533188 0.063355 rpy=3.3411E-05 1.5707 2.618
- joint wheel2_joint: origin xyz=-0.0014342 -0.15301 0.063355 rpy=1.5708 1.5708 0 -> xyz=-0.001402062 -0.149010130 0.063355 rpy=1.5708 1.5708 0
- joint wheel3_joint: origin xyz=0.13115 0.076408 0.063355 rpy=-1.5708 0 -1.0472 -> xyz=0.127692644 0.074396362 0.063355 rpy=-1.5708 0 -1.0472

File: src/alohamini_description/urdf/alohamini2pro_moveit.urdf (robot description, URDF)
Before this commit: robot alohamini2pro_moveit, 31 links, 30 joints
Links:
- link wheel1: geometry collision cylinder length=0.0510028 radius=0.0634601; visual mesh filename=package://alohamini_description/meshes/visual/Link2_dp.STL
- link wheel2: geometry collision cylinder length=0.0510001 radius=0.0634601; visual mesh filename=package://alohamini_description/meshes/visual/Link3_dp.STL
- link wheel3: geometry collision cylinder length=0.0510001 radius=0.0634609; visual mesh filename=package://alohamini_description/meshes/visual/Link4_dp.STL
Joints:
- joint wheel1_joint: origin xyz=-0.1337 0.076522 0.063355 rpy=3.3411E-05 1.5707 2.618 -> xyz=-0.130229464 0.074533188 0.063355 rpy=3.3411E-05 1.5707 2.618
- joint wheel2_joint: origin xyz=-0.0014342 -0.15301 0.063355 rpy=1.5708 1.5708 0 -> xyz=-0.001402062 -0.149010130 0.063355 rpy=1.5708 1.5708 0
- joint wheel3_joint: origin xyz=0.13115 0.076408 0.063355 rpy=-1.5708 0 -1.0472 -> xyz=0.127692644 0.074396362 0.063355 rpy=-1.5708 0 -1.0472

Commit message: feat: add guarded trajectory action bridge

File: src/alohamini_description/urdf/alohamini2pro_kinematic.urdf (robot description, URDF)
Before this commit: robot alohamini2pro_kinematic, 31 links, 30 joints
Joints:
- joint left_shoulder_pan: limit lower=-2.13376727595 upper=2.23961195031 effort=1.57 velocity=4.2 -> lower=-2.23961195031 upper=2.13376727595 effort=1.57 velocity=4.2
- joint left_wrist_yaw_joint: limit lower=-1.24559239976 upper=1.19190307219 effort=1.57 velocity=4.2 -> lower=-0.978679742671 upper=1.45881572928 effort=1.57 velocity=4.2
- joint right_shoulder_pan: limit lower=-2.13376727595 upper=2.23961195031 effort=1.57 velocity=4.2 -> lower=-2.23961195031 upper=2.13376727595 effort=1.57 velocity=4.2
- joint right_wrist_yaw_joint: limit lower=-1.24559239976 upper=1.19190307219 effort=1.57 velocity=4.2 -> lower=-0.978679742671 upper=1.45881572928 effort=1.57 velocity=4.2

File: src/alohamini_description/urdf/alohamini2pro_left_kinematic.urdf (robot description, URDF)
Before this commit: robot alohamini2pro_left_kinematic, 10 links, 9 joints
Joints:
- joint left_shoulder_pan: limit lower=-2.13376727595 upper=2.23961195031 effort=1.57 velocity=4.2 -> lower=-2.23961195031 upper=2.13376727595 effort=1.57 velocity=4.2
- joint left_wrist_yaw_joint: limit lower=-1.24559239976 upper=1.19190307219 effort=1.57 velocity=4.2 -> lower=-0.978679742671 upper=1.45881572928 effort=1.57 velocity=4.2

File: src/alohamini_description/urdf/alohamini2pro_moveit.urdf (robot description, URDF)
Before this commit: robot alohamini2pro_moveit, 31 links, 30 joints
Joints:
- joint left_shoulder_pan: limit lower=-2.13376727595 upper=2.23961195031 effort=1.57 velocity=4.2 -> lower=-2.23961195031 upper=2.13376727595 effort=1.57 velocity=4.2
- joint left_wrist_yaw_joint: limit lower=-1.24559239976 upper=1.19190307219 effort=1.57 velocity=4.2 -> lower=-0.978679742671 upper=1.45881572928 effort=1.57 velocity=4.2
- joint right_shoulder_pan: limit lower=-2.13376727595 upper=2.23961195031 effort=1.57 velocity=4.2 -> lower=-2.23961195031 upper=2.13376727595 effort=1.57 velocity=4.2
- joint right_wrist_yaw_joint: limit lower=-1.24559239976 upper=1.19190307219 effort=1.57 velocity=4.2 -> lower=-0.978679742671 upper=1.45881572928 effort=1.57 velocity=4.2

File: src/alohamini_description/urdf/alohamini2pro_right_kinematic.urdf (robot description, URDF)
Before this commit: robot alohamini2pro_right_kinematic, 10 links, 9 joints
Joints:
- joint right_shoulder_pan: limit lower=-2.13376727595 upper=2.23961195031 effort=1.57 velocity=4.2 -> lower=-2.23961195031 upper=2.13376727595 effort=1.57 velocity=4.2
- joint right_wrist_yaw_joint: limit lower=-1.24559239976 upper=1.19190307219 effort=1.57 velocity=4.2 -> lower=-0.978679742671 upper=1.45881572928 effort=1.57 velocity=4.2

Commit message: 左右臂标定+凸碰撞箱

File: src/alohamini_description/urdf/alohamini2pro_kinematic.urdf (robot description, URDF)
Before this commit: robot alohamini2pro_kinematic, 31 links, 30 joints
Joints:
- joint left_elbow_flex: limit lower=-0.0703594430376 upper=3.22002934698 effort=2.21 velocity=2.48 -> lower=-0.010737865514856 upper=3.258175193469144 effort=2.21 velocity=2.48
- joint left_shoulder_lift: limit lower=-3.29519440558 upper=0.160864309523 effort=2.21 velocity=2.48 -> lower=-3.505146100318774 upper=0.018407769454226 effort=2.21 velocity=2.48
- joint left_shoulder_pan: limit lower=-2.23961195031 upper=2.13376727595 effort=1.57 velocity=4.2 -> lower=-2.196660488252487 upper=2.208932334555513 effort=1.57 velocity=4.2
- joint left_wrist_flex: limit lower=-1.6459613854 upper=1.48335942189 effort=1.57 velocity=4.2 -> lower=-1.776349752372000 upper=1.524776903158000 effort=1.57 velocity=4.2
- joint left_wrist_yaw_joint: limit lower=-0.978679742671 upper=1.45881572928 effort=1.57 velocity=4.2 -> lower=-1.437339998248976 upper=1.529378845522024 effort=1.57 velocity=4.2
- joint right_elbow_flex: limit lower=-0.0703594430376 upper=3.22002934698 effort=2.21 velocity=2.48 -> lower=-0.012271846303223 upper=3.330272290499778 effort=2.21 velocity=2.48
- joint right_shoulder_lift: limit lower=-3.29519440558 upper=0.160864309523 effort=2.21 velocity=2.48 -> lower=-3.482136388500722 upper=0.009203884727279 effort=2.21 velocity=2.48
- joint right_shoulder_pan: limit lower=-2.23961195031 upper=2.13376727595 effort=1.57 velocity=4.2 -> lower=-2.219670200070399 upper=2.184388641949601 effort=1.57 velocity=4.2
- joint right_wrist_flex: limit lower=-1.6459613854 upper=1.48335942189 effort=1.57 velocity=4.2 -> lower=-1.669204307772067 upper=1.582834962545933 effort=1.57 velocity=4.2
- joint right_wrist_yaw_joint: limit lower=-0.978679742671 upper=1.45881572928 effort=1.57 velocity=4.2 -> lower=-1.477223498733657 upper=1.475689517946343 effort=1.57 velocity=4.2

File: src/alohamini_description/urdf/alohamini2pro_left_kinematic.urdf (robot description, URDF)
Before this commit: robot alohamini2pro_left_kinematic, 10 links, 9 joints
Joints:
- joint left_elbow_flex: limit lower=-0.0703594430376 upper=3.22002934698 effort=2.21 velocity=2.48 -> lower=-0.010737865514856 upper=3.258175193469144 effort=2.21 velocity=2.48
- joint left_shoulder_lift: limit lower=-3.29519440558 upper=0.160864309523 effort=2.21 velocity=2.48 -> lower=-3.505146100318774 upper=0.018407769454226 effort=2.21 velocity=2.48
- joint left_shoulder_pan: limit lower=-2.23961195031 upper=2.13376727595 effort=1.57 velocity=4.2 -> lower=-2.196660488252487 upper=2.208932334555513 effort=1.57 velocity=4.2
- joint left_wrist_flex: limit lower=-1.6459613854 upper=1.48335942189 effort=1.57 velocity=4.2 -> lower=-1.776349752372000 upper=1.524776903158000 effort=1.57 velocity=4.2
- joint left_wrist_yaw_joint: limit lower=-0.978679742671 upper=1.45881572928 effort=1.57 velocity=4.2 -> lower=-1.437339998248976 upper=1.529378845522024 effort=1.57 velocity=4.2

File: src/alohamini_description/urdf/alohamini2pro_moveit.urdf (robot description, URDF)
Before this commit: robot alohamini2pro_moveit, 31 links, 30 joints
Links:
- link left_Base: geometry collision mesh filename=package://alohamini_description/meshes/collision/arm_base_v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; visual mesh filename=package://alohamini_description/meshes/visual/left_Base.STL
- link left_Fixed_Jaw: geometry collision mesh filename=package://alohamini_description/meshes/collision/fixed_jaw_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; visual mesh filename=package://alohamini_description/meshes/visual/left_Fixed_Ja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
- link left_Lower_Arm: geometry collision mesh filename=package://alohamini_description/meshes/collision/lower_arm_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; visual mesh filename=package://alohamini_description/meshes/visual/left_Lower_Ar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
- link left_Rotation_Pitch: geometry collision mesh filename=package://alohamini_description/meshes/collision/rotation_p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; visual mesh filename=package://alohamini_description/meshes/visual/left_Rotation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
- link left_Upper_Arm: geometry collision mesh filename=package://alohamini_description/meshes/collision/upper_arm_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; visual mesh filename=package://alohamini_description/meshes/visual/left_Upper_Ar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
- link left_Wrist_Pitch_Roll: geometry collision mesh filename=package://alohamini_description/meshes/collision/wrist_pitc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; visual mesh filename=package://alohamini_description/meshes/visual/left_Wrist_Pi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
- link left_camera: geometry collision mesh filename=package://alohamini_description/meshes/collision/wrist_came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; visual mesh filename=package://alohamini_description/meshes/visual/left_camera.S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
- link left_wrist_yaw: geometry collision mesh filename=package://alohamini_description/meshes/collision/wrist_yaw_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; visual mesh filename=package://alohamini_description/meshes/visual/left_wrist_ya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
- link right_Base: geometry collision mesh filename=package://alohamini_description/meshes/collision/arm_base_v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; visual mesh filename=package://alohamini_description/meshes/visual/right_Base.STL
- link right_Fixed_Jaw: geometry collision mesh filename=package://alohamini_description/meshes/collision/fixed_jaw_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; visual mesh filename=package://alohamini_description/meshes/visual/right_Fixed_J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
- link right_Lower_Arm: geometry collision mesh filename=package://alohamini_description/meshes/collision/lower_arm_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; visual mesh filename=package://alohamini_description/meshes/visual/right_Lower_A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
- link right_Rotation_Pitch: geometry collision mesh filename=package://alohamini_description/meshes/collision/rotation_p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; visual mesh filename=package://alohamini_description/meshes/visual/right_Rotatio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
- link right_Upper_Arm: geometry collision mesh filename=package://alohamini_description/meshes/collision/upper_arm_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; visual mesh filename=package://alohamini_description/meshes/visual/right_Upper_A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
- link right_Wrist_Pitch_Roll: geometry collision mesh filename=package://alohamini_description/meshes/collision/wrist_pitc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; visual mesh filename=package://alohamini_description/meshes/visual/right_Wrist_P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
- link right_camera: geometry collision mesh filename=package://alohamini_description/meshes/collision/wrist_came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; visual mesh filename=package://alohamini_description/meshes/visual/right_camera.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
- link right_wrist_yaw: geometry collision mesh filename=package://alohamini_description/meshes/collision/wrist_yaw_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; visual mesh filename=package://alohamini_description/meshes/visual/right_wrist_y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
Joints:
- joint left_elbow_flex: limit lower=-0.0703594430376 upper=3.22002934698 effort=2.21 velocity=2.48 -> lower=-0.010737865514856 upper=3.258175193469144 effort=2.21 velocity=2.48
- joint left_shoulder_lift: limit lower=-3.29519440558 upper=0.160864309523 effort=2.21 velocity=2.48 -> lower=-3.505146100318774 upper=0.018407769454226 effort=2.21 velocity=2.48
- joint left_shoulder_pan: limit lower=-2.23961195031 upper=2.13376727595 effort=1.57 velocity=4.2 -> lower=-2.196660488252487 upper=2.208932334555513 effort=1.57 velocity=4.2
- joint left_wrist_flex: limit lower=-1.6459613854 upper=1.48335942189 effort=1.57 velocity=4.2 -> lower=-1.776349752372000 upper=1.524776903158000 effort=1.57 velocity=4.2
- joint left_wrist_yaw_joint: limit lower=-0.978679742671 upper=1.45881572928 effort=1.57 velocity=4.2 -> lower=-1.437339998248976 upper=1.529378845522024 effort=1.57 velocity=4.2
- joint right_elbow_flex: limit lower=-0.0703594430376 upper=3.22002934698 effort=2.21 velocity=2.48 -> lower=-0.012271846303223 upper=3.330272290499778 effort=2.21 velocity=2.48
- joint right_shoulder_lift: limit lower=-3.29519440558 upper=0.160864309523 effort=2.21 velocity=2.48 -> lower=-3.482136388500722 upper=0.009203884727279 effort=2.21 velocity=2.48
- joint right_shoulder_pan: limit lower=-2.23961195031 upper=2.13376727595 effort=1.57 velocity=4.2 -> lower=-2.219670200070399 upper=2.184388641949601 effort=1.57 velocity=4.2
- joint right_wrist_flex: limit lower=-1.6459613854 upper=1.48335942189 effort=1.57 velocity=4.2 -> lower=-1.669204307772067 upper=1.582834962545933 effort=1.57 velocity=4.2
- joint right_wrist_yaw_joint: limit lower=-0.978679742671 upper=1.45881572928 effort=1.57 velocity=4.2 -> lower=-1.477223498733657 upper=1.475689517946343 effort=1.57 velocity=4.2

File: src/alohamini_description/urdf/alohamini2pro_right_kinematic.urdf (robot description, URDF)
Before this commit: robot alohamini2pro_right_kinematic, 10 links, 9 joints
Joints:
- joint right_elbow_flex: limit lower=-0.0703594430376 upper=3.22002934698 effort=2.21 velocity=2.48 -> lower=-0.012271846303223 upper=3.330272290499778 effort=2.21 velocity=2.48
- joint right_shoulder_lift: limit lower=-3.29519440558 upper=0.160864309523 effort=2.21 velocity=2.48 -> lower=-3.482136388500722 upper=0.009203884727279 effort=2.21 velocity=2.48
- joint right_shoulder_pan: limit lower=-2.23961195031 upper=2.13376727595 effort=1.57 velocity=4.2 -> lower=-2.219670200070399 upper=2.184388641949601 effort=1.57 velocity=4.2
- joint right_wrist_flex: limit lower=-1.6459613854 upper=1.48335942189 effort=1.57 velocity=4.2 -> lower=-1.669204307772067 upper=1.582834962545933 effort=1.57 velocity=4.2
- joint right_wrist_yaw_joint: limit lower=-0.978679742671 upper=1.45881572928 effort=1.57 velocity=4.2 -> lower=-1.477223498733657 upper=1.475689517946343 effort=1.57 velocity=4.2

Commit message: 修正了baselink坐标系

File: src/alohamini_description/urdf/alohamini2pro_kinematic.urdf (robot description, URDF)
Before this commit: robot alohamini2pro_kinematic, 31 links, 30 joints
Links:
- added link base_cad_link
Joints:
- added joint base_cad_joint: type fixed, parent base_link, child base_cad_link, origin xyz=0 0 0 rpy=0 0 1.5707963267948966
- joint back_camera_joint5_dp: parent base_link -> base_cad_link
- joint front_camera_joint6_dp: parent base_link -> base_cad_link
- joint vertical_move: parent base_link -> base_cad_link
- joint wheel1_joint: parent base_link -> base_cad_link
- joint wheel2_joint: parent base_link -> base_cad_link
- joint wheel3_joint: parent base_link -> base_cad_link

File: src/alohamini_description/urdf/alohamini2pro_moveit.urdf (robot description, URDF)
Before this commit: robot alohamini2pro_moveit, 31 links, 30 joints
Links:
- added link base_cad_link, mass 9.6; collision mesh filename=package://alohamini_description/meshes/visual/base_link.STL; visual mesh filename=package://alohamini_description/meshes/visual/base_link.STL
- link base_link: mass 9.6 -> None; geometry 
Joints:
- added joint base_cad_joint: type fixed, parent base_link, child base_cad_link, origin xyz=0 0 0 rpy=0 0 1.5707963267948966
- joint back_camera_joint5_dp: parent base_link -> base_cad_link
- joint front_camera_joint6_dp: parent base_link -> base_cad_link
- joint vertical_move: parent base_link -> base_cad_link
- joint wheel1_joint: parent base_link -> base_cad_link
- joint wheel2_joint: parent base_link -> base_cad_link
- joint wheel3_joint: parent base_link -> base_cad_link
