Commit message: 修改了夹爪碰撞+gazebo demo

File: src/alohamini_description/urdf/alohamini2pro_moveit.urdf (robot description, URDF)
Before this commit: robot alohamini2pro_moveit, 32 links, 31 joints
Links:
- link left_Fixed_Jaw: geometry collision box size=0.010 0.014 0.064; collision mesh filename=package://alohamini_description/meshes/collision/fixed_jaw_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
- link left_Moving_Jaw: geometry collision box size=0.010 0.014 0.064; collision mesh filename=package://alohamini_description/meshes/collision/moving_jaw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
- link right_Fixed_Jaw: geometry collision box size=0.010 0.014 0.064; collision mesh filename=package://alohamini_description/meshes/collision/fixed_jaw_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
- link right_Moving_Jaw: geometry collision box size=0.010 0.014 0.064; collision mesh filename=package://alohamini_description/meshes/collision/moving_jaw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

File: src/alohamini_description/urdf/source/alohamini2pro_cad.urdf (robot description, URDF)
Before this commit: robot alohamini2pro_urdf, 29 links, 28 joints
Links:
- link left_Fixed_Jaw: geometry collision box size=0.010 0.014 0.064; collision mesh filename=package://alohamini_description/meshes/collision/fixed_jaw_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
- link left_Moving_Jaw: geometry collision box size=0.010 0.014 0.064; collision mesh filename=package://alohamini_description/meshes/collision/moving_jaw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
- link right_Fixed_Jaw: geometry collision box size=0.010 0.014 0.064; collision mesh filename=package://alohamini_description/meshes/collision/fixed_jaw_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
- link right_Moving_Jaw: geometry collision box size=0.010 0.014 0.064; collision mesh filename=package://alohamini_description/meshes/collision/moving_jaw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

File: src/alohamini_description/urdf/source/alohamini2pro_right_arm.urdf (robot description, URDF)
Before this commit: robot alohamini2pro_right_arm, 9 links, 8 joints
Links:
- link right_Fixed_Jaw: geometry collision box size=0.010 0.014 0.064; collision mesh filename=package://alohamini_description/meshes/collision/fixed_jaw_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
- link right_Moving_Jaw: geometry collision box size=0.010 0.014 0.064; collision mesh filename=package://alohamini_description/meshes/collision/moving_jaw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
